File: motoco.sch (KiCad schematic (older format))
At the start: 12 parts, among them M1 Motor_DC, Q1 Q_PMOS_SGD, Q2 Q_NMOS_SGD, Q3 Q_PMOS_SGD, Q4 Q_NMOS_SGD, U1 SFH617A-1, U2 SFH617A-1

Commit message: update
Parts:
- removed Q1, Q3: Q_PMOS_SGD, symbol Device:Q_PMOS_SGD
- removed Q4: Q_NMOS_SGD, symbol Device:Q_NMOS_SGD
- removed U1, U2: SFH617A-1, Package_DIP:DIP-4_W7.62mm, symbol Isolator:SFH617A-1
- added CC1, CSNH1: C, symbol Device:C
- added D?: DIODE, symbol pspice:DIODE
- added SNH1: R, symbol Device:R
- added U3: TLE7182EM, Package_SO:SSOP-24_3.9x8.7mm_P0.635mm, symbol tle7182em:TLE7182EM
- renumbered Q2 to Q1, R1 to RGH1
Connections:
- net labels added: GNDPWR
- net labels removed: DIO1
- wire segments 28 -> 35
Other:
- moved on the sheet: C1, M1, Q1, R2, R3, R4, RGH1

Commit message: update
Parts:
- added C12: 100p, symbol Device:C
- added C14, C15: 10p, symbol Device:C
- added C16, C17: 220p, symbol Device:C
- added C18, C20: 2,2uF/50V, symbol Device:C
- added C19, C4: 100n, symbol Device:C
- added C24, C?: C, symbol Device:C
- added C26, C28: 220u/50V, symbol Device:CP
- added C29, C?: 2,2nF, symbol Device:C
- added C3, C6, C9: 4,7nF, symbol Device:C
- added C5: 2,2u, symbol Device:C
- added C7, C8: 330n, symbol Device:C
- added D1, D3, D5, D6, D8: D, symbol Device:D
- added D? (x4): BAW56DW, Package_TO_SOT_SMD:SOT-363_SC-70-6, symbol Diode:BAW56DW
- added D?: D_Zener, symbol Device:D_Zener
- added HS1, LS1, LS2, RPP-MOSFET: IPD90N04S4-02, symbol Device:Q_NMOS_SGD
- added L?: L, symbol Device:L
- added Q?: Q_NPN_BCE, symbol Device:Q_NPN_BCE
- added R10, R11, R9: 0R, symbol Device:R
- added R12, R13: 220R 1%, symbol Device:R
- added R14, R15, R16, R44: 10K 1%, symbol Device:R
- added R17: 1K, symbol Device:R
- added R18: 4k7, symbol Device:R
- added R19: 22R 1%, symbol Device:R
- added R2, R3: 2,2R, symbol Device:R
- added R22: 1R, symbol Device:R
- added R43: 47K, symbol Device:R
- added R5, R6, R7, R8: 10R 1%, symbol Device:R
- added R? (x3): R, symbol Device:R
- HS2: renamed from Q1; value Q_NMOS_SGD -> IPD90N04S4-02
Connections:
- net labels added: +5V, OUT1, OUT2
- wire segments 35 -> 214
Other:
- moved on the sheet: C1, CC1, CSNH1, D?, HS2, M1, R2, R3, R4, RGH1, SNH1, U3
