File: ver1/motoco.sch (KiCad schematic (older format))
At the start: 72 parts, among them M1 Motor_DC, U3 TLE7182EM

Commit message: update
Parts:
- removed C1, CC1, CSNH1: C, symbol Device:C
- removed D?: DIODE, symbol pspice:DIODE
- removed R2, R3, R4, RGH1, SNH1: R, symbol Device:R
- added C21: 100n, symbol Device:C
- added C22, C23: 22n, symbol Device:C
- added ERR: LED, symbol Device:LED
- added FAB32Q2_A, FAB32Q2_B: Conn_01x16_Female, symbol Connector:Conn_01x16_Female
- added GMSTBA5: Conn_01x05_Female, symbol Connector:Conn_01x05_Female
- added JP1, JP2, JP3, JP4, JP5: Conn_01x02_Female, symbol Connector:Conn_01x02_Female
- added R20: 100K, symbol Device:R_POT_US
- added R23: 22K, symbol Device:R
- added R24: 1K, symbol Device:R
- added R25: 50K, symbol Device:R_POT_US
- added R27, R29, R30, R32, R34, R35, R36: 10K, symbol Device:R
- added R31: 200K, symbol Device:R_POT_US
- added R38: 2k7, symbol Device:R
- added R39, R42: 47K, symbol Device:R
- added R40, R41: 5,1K, symbol Device:R
- added R?: R, symbol Device:R
- added RESET: SW_Push, symbol Switch:SW_Push
- added SJ2, SJ3, SJ4: SolderJumper_3_Open, symbol Jumper:SolderJumper_3_Open
Connections:
- net labels added: DRV, ERR, IH1, IH2, IL1, IL2, ISO*, PWM
- net labels removed: DIO2, VCCQ
- wire segments 214 -> 296
Other:
- note added: "ADD 5V REG HERE"
- moved on the sheet: M1, R17
