File: ver2/hardware/motoco.sch (KiCad schematic (older format))
At the start: 95 parts, among them M1 Motor_DC, U3 TLE7182EM

Commit message: update
Parts:
- removed Q?: Q_NPN_BCE, symbol Device:Q_NPN_BCE
- added C10: 22u/50V, symbol Device:CP
- added C11: 10u, symbol Device:C
- added C13: 47n/50V, symbol Device:C
- added D9: 5V, symbol Device:LED
- added Q1: BC846B, Package_TO_SOT_SMD:SOT-23, symbol Device:Q_NPN_BEC
- added R21: 1R, symbol Device:R
- added R37: 2k7, symbol Device:R
- added U1: TLE4269G, symbol tle4269g:TLE4269G
- C1: renamed from C?; value 2,2nF -> 4,7nF
- D7: renamed from D?; value D_Zener -> ZMM12
- R1: renamed from R?; value R -> 2,2R
- gave numbers to parts that had none: 5
- renumbered ERR to ERR1, FAB32Q2_A to FAB32Q2_A1, FAB32Q2_B to FAB32Q2_B1, RESET to RESET1, RPP-MOSFET to RPP-MOSFET1
Connections:
- net +5V: now also C11.2, D9.2 (A), U1.8 (Q)
- net GND: now also C10.2, C11.1, C13.1, R37.2, U1.5 (GND)
- net at C1.1, C26.1, C28.1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: now also R22.1, R21.1
- net at R18.2, U3.6 (RPP): no longer R22.1
- net at R18.1, RPP-MOSFET1.2 (G): now also Q1.3 (C)
- net at RPP-MOSFET1.1 (S): now also D7.1 (K), L1.1
- net at R43.1: now also Q1.1 (B)
- net at D7.2 (A): now also Q1.2 (E)
- new net: C10.1, C13.2, R21.2, U1.1 (I)
- new net: D9.1 (K), R37.1
Other:
- note removed: "ADD 5V REG HERE"
- note removed: "Low-side N-FET #1"

Commit message: update
Parts:
- removed HS1, HS2, LS1, LS2, RPP-MOSFET1: IPD90N04S4-02, symbol Device:Q_NMOS_SGD
- added HS1, HS2, LS1, LS2, RPP-MOSFET1: IPD90N04S4-02, footprints:PG-TO-252-3-313, symbol Device:Q_NMOS_GDS
- C1, C11, C12, C13, C14, C15, C16, C17, C18, C19, C20, C21, C22, C23, C29, C3, C4, C5, C6, C7, C8, C9: footprint (none) -> Capacitor_SMD:C_0805_2012Metric_Pad1.15x1.40mm_HandSolder
- C10: footprint (none) -> Capacitor_THT:CP_Radial_D5.0mm_P2.00mm
- C2: value C -> 100nF; footprint (none) -> Capacitor_SMD:C_0805_2012Metric_Pad1.15x1.40mm_HandSolder
- C24: value C -> (n.m.); footprint (none) -> Capacitor_SMD:C_0805_2012Metric_Pad1.15x1.40mm_HandSolder
- C26, C28: footprint (none) -> Capacitor_THT:CP_Radial_D16.0mm_P7.50mm
- D1, D3, D5, D6, D8: footprint (none) -> Diode_SMD:D_0805_2012Metric
- D2, D4: footprint (none) -> Package_TO_SOT_SMD:SOT-23
- D7: footprint (none) -> Diode_SMD:D_MiniMELF_Handsoldering
- D9, ERR1: footprint (none) -> LED_SMD:LED_0805_2012Metric_Pad1.15x1.40mm_HandSolder
- L1: value L -> SER2011-202; footprint (none) -> footprints:SER2011-202-REAL
- R1, R10, R11, R12, R13, R14, R15, R16, R17, R18, R19, R2, R20, R21, R22, R23, R24, R25, R26, R27, R28, R29, R3, R30, R31, R32, R34, R35, R36, R37, R38, R39, R4, R40, R41, R42, R43, R44, R5, R6, R7, R8, R9: footprint (none) -> Resistor_SMD:R_0805_2012Metric_Pad1.15x1.40mm_HandSolder
- U1: footprint (none) -> Package_SO:Infineon_PG-DSO-8-43
- U3: footprint Package_SO:SSOP-24_3.9x8.7mm_P0.635mm -> footprints:PG-SSOP-24-9
Connections:
- net OUT1: now also HS1.3 (S), LS1.2 (D)
- net OUT2: now also HS2.3 (S), LS2.2 (D)
- net at D3.2 (A), R5.1: now also HS2.1 (G)
- net at C1.1, C26.1, C28.1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: now also HS1.2 (D), HS2.2 (D), RPP-MOSFET1.2 (D)
- net at D6.2 (A), R7.1: now also LS1.1 (G)
- net at D8.2 (A), R8.1: now also LS2.1 (G)
- net at C24.2, R11.1, R12.1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: now also LS1.3 (S), LS2.3 (S)
- net at D1.2 (A), R6.1: now also HS1.1 (G)
- net at Q1.3 (C), R18.1: now also RPP-MOSFET1.1 (G)
- net at D7.1 (K), L1.1: now also RPP-MOSFET1.3 (S)

Commit message: update
Parts:
- FAB32Q2_A1, FAB32Q2_B1: footprint (none) -> Connector_PinSocket_2.54mm:PinSocket_1x16_P2.54mm_Vertical
- GMSTBA5: footprint (none) -> Connector_PinSocket_2.54mm:PinSocket_1x05_P2.54mm_Vertical
- JP1, JP2, JP3, JP4, JP5: footprint (none) -> Connector_PinSocket_2.54mm:PinSocket_1x02_P2.54mm_Vertical
- M1: footprint (none) -> TerminalBlock_Phoenix:TerminalBlock_Phoenix_MKDS-1,5-2_1x02_P5.00mm_Horizontal
- RESET1: footprint (none) -> Button_Switch_SMD:SW_Push_1P1T_NO_6x6mm_H9.5mm
- SJ2, SJ3, SJ4: footprint (none) -> Jumper:SolderJumper-3_P1.3mm_Open_Pad1.0x1.5mm
Changed lines of the file:
@@
 F 0 "M1" V 20345 6650 50  0000 C CNN
 F 1 "Motor_DC" V 20254 6650 50  0000 C CNN
-F 2 "" H 20050 6610 50  0001 C CNN
+F 2 "TerminalBlock_Phoenix:TerminalBlock_Phoenix_MKDS-1,5-2_1x02_P5.00mm_Horizontal" H 20050 6610 50  0001 C CNN
 F 3 "~" H 20050 6610 50  0001 C CNN
 	1    20050 6700
@@
 F 0 "JP1" V 10488 6862 50  0000 R CNN
 F 1 "Conn_01x02_Female" V 10250 7150 50  0001 R CNN
-F 2 "" H 10550 7050 50  0001 C CNN
+F 2 "Connector_PinSocket_2.54mm:PinSocket_1x02_P2.54mm_Vertical" H 10550 7050 50  0001 C CNN
 F 3 "~" H 10550 7050 50  0001 C CNN
 	1    10550 7050
@@
 F 0 "JP5" V 8488 6462 50  0000 R CNN
 F 1 "Conn_01x02_Female" V 8300 6950 50  0001 R CNN
-F 2 "" H 8550 6650 50  0001 C CNN
+F 2 "Connector_PinSocket_2.54mm:PinSocket_1x02_P2.54mm_Vertical" H 8550 6650 50  0001 C CNN
 F 3 "~" H 8550 6650 50  0001 C CNN
 	1    8550 6650
@@
 F 0 "RESET1" V 9504 9498 50  0000 L CNN
 F 1 "SW_Push" V 9595 9498 50  0000 L CNN
-F 2 "" H 9550 9550 50  0001 C CNN
+F 2 "Button_Switch_SMD:SW_Push_1P1T_NO_6x6mm_H9.5mm" H 9550 9550 50  0001 C CNN
 F 3 "~" H 9550 9550 50  0001 C CNN
 	1    9550 9350
@@
 F 0 "JP3" V 8500 7350 50  0000 R CNN
 F 1 "Conn_01x02_Female" V 8700 7450 50  0001 R CNN
-F 2 "" H 8600 7100 50  0001 C CNN
+F 2 "Connector_PinSocket_2.54mm:PinSocket_1x02_P2.54mm_Vertical" H 8600 7100 50  0001 C CNN
 F 3 "~" H 8600 7100 50  0001 C CNN
 	1    8600 7100
@@
 F 0 "JP2" V 10138 8212 50  0000 R CNN
 F 1 "Conn_01x02_Female" V 10300 8750 50  0001 R CNN
-F 2 "" H 10200 8400 50  0001 C CNN
+F 2 "Connector_PinSocket_2.54mm:PinSocket_1x02_P2.54mm_Vertical" H 10200 8400 50  0001 C CNN
 F 3 "~" H 10200 8400 50  0001 C CNN
 	1    10200 8400
@@
 F 0 "JP4" V 8838 8212 50  0000 R CNN
 F 1 "Conn_01x02_Female" V 9000 8750 50  0001 R CNN
-F 2 "" H 8900 8400 50  0001 C CNN
+F 2 "Connector_PinSocket_2.54mm:PinSocket_1x02_P2.54mm_Vertical" H 8900 8400 50  0001 C CNN
 F 3 "~" H 8900 8400 50  0001 C CNN
 	1    8900 8400
@@
 F 0 "SJ4" V 7500 8867 50  0000 L CNN
 F 1 "SolderJumper_3_Open" V 7455 8867 50  0001 L CNN
-F 2 "" H 7500 8800 50  0001 C CNN
+F 2 "Jumper:SolderJumper-3_P1.3mm_Open_Pad1.0x1.5mm" H 7500 8800 50  0001 C CNN
 F 3 "~" H 7500 8800 50  0001 C CNN
 	1    7500 8800
@@
 F 0 "SJ3" V 7700 8317 50  0000 L CNN
 F 1 "SolderJumper_3_Open" V 7655 8317 50  0001 L CNN
-F 2 "" H 7700 8250 50  0001 C CNN
+F 2 "Jumper:SolderJumper-3_P1.3mm_Open_Pad1.0x1.5mm" H 7700 8250 50  0001 C CNN
 F 3 "~" H 7700 8250 50  0001 C CNN
 	1    7700 8250
@@
 F 0 "SJ2" V 8200 8017 50  0000 L CNN
 F 1 "SolderJumper_3_Open" V 8245 8017 50  0001 L CNN
-F 2 "" H 8200 7950 50  0001 C CNN
+F 2 "Jumper:SolderJumper-3_P1.3mm_Open_Pad1.0x1.5mm" H 8200 7950 50  0001 C CNN
 F 3 "~" H 8200 7950 50  0001 C CNN
 	1    8200 7950
@@
 F 0 "FAB32Q2_B1" H 4692 8885 50  0000 C CNN
 F 1 "Conn_01x16_Female" H 4692 8794 50  0001 C CNN
-F 2 "" H 4800 8000 50  0001 C CNN
+F 2 "Connector_PinSocket_2.54mm:PinSocket_1x16_P2.54mm_Vertical" H 4800 8000 50  0001 C CNN
 F 3 "~" H 4800 8000 50  0001 C CNN
 	1    4800 8000
@@
 F 0 "FAB32Q2_A1" H 2642 8993 50  0000 C CNN
 F 1 "Conn_01x16_Female" H 2642 8994 50  0001 C CNN
-F 2 "" H 2750 8200 50  0001 C CNN
+F 2 "Connector_PinSocket_2.54mm:PinSocket_1x16_P2.54mm_Vertical" H 2750 8200 50  0001 C CNN
 F 3 "~" H 2750 8200 50  0001 C CNN
 	1    2750 8200
@@
 F 0 "GMSTBA5" H 9892 3843 50  0000 C CNN
 F 1 "Conn_01x05_Female" H 9892 3844 50  0001 C CNN
-F 2 "" H 10000 3550 50  0001 C CNN
+F 2 "Connector_PinSocket_2.54mm:PinSocket_1x05_P2.54mm_Vertical" H 10000 3550 50  0001 C CNN
 F 3 "~" H 10000 3550 50  0001 C CNN
 	1    10000 3550

Commit message: update
Parts:
- renumbered U3 to IC1, U1 to IC2
Changed lines of the file:
@@
 $EndComp
 $Comp
-L tle7182em:TLE7182EM U3
+L tle7182em:TLE7182EM IC1
 U 1 1 5F26DA69
 P 11900 7750
-F 0 "U3" H 12100 6600 50  0000 C CNN
+F 0 "IC1" H 12100 6600 50  0000 C CNN
 F 1 "TLE7182EM" V 11900 8050 50  0000 C CNN
 F 2 "footprints:PG-SSOP-24-9" H 11900 8050 50  0001 C CNN
@@
 	11700 4000 15100 4000
 $Comp
-L tle4269g:TLE4269G U1
+L tle4269g:TLE4269G IC2
 U 1 1 5F54667B
 P 8750 5300
-F 0 "U1" H 8775 5865 50  0000 C CNN
+F 0 "IC2" H 8775 5865 50  0000 C CNN
 F 1 "TLE4269G" H 8775 5774 50  0000 C CNN
 F 2 "Package_SO:Infineon_PG-DSO-8-43" H 8750 5300 50  0001 C CNN

Commit message: update
Parts:
- C1, C11, C12, C14, C15, C16, C17, C19, C2, C21, C22, C23, C24, C3, C4, C6, C7, C8, C9: footprint Capacitor_SMD:C_0805_2012Metric_Pad1.15x1.40mm_HandSolder -> Capacitor_SMD:C_0603_1608Metric_Pad1.05x0.95mm_HandSolder
- C13, C29: footprint Capacitor_SMD:C_0805_2012Metric_Pad1.15x1.40mm_HandSolder -> Capacitor_SMD:C_1210_3225Metric
- C18, C20: footprint Capacitor_SMD:C_0805_2012Metric_Pad1.15x1.40mm_HandSolder -> Capacitor_SMD:C_1206_3216Metric
- C5: footprint Capacitor_SMD:C_0805_2012Metric_Pad1.15x1.40mm_HandSolder -> Capacitor_SMD:C_1210_3225Metric_Pad1.42x2.65mm_HandSolder
- D1, D3, D5, D6, D8: footprint Diode_SMD:D_0805_2012Metric -> Diode_SMD:D_MiniMELF_Handsoldering
- D9, ERR1: footprint LED_SMD:LED_0805_2012Metric_Pad1.15x1.40mm_HandSolder -> LED_SMD:LED_0603_1608Metric_Pad1.05x0.95mm_HandSolder
- R1, R2, R3, R37, R38, R4: footprint Resistor_SMD:R_0805_2012Metric_Pad1.15x1.40mm_HandSolder -> Resistor_SMD:R_1206_3216Metric
- R10, R11, R12, R13, R14, R15, R16, R17, R18, R19, R21, R22, R23, R24, R26, R27, R28, R29, R30, R32, R34, R35, R36, R39, R40, R41, R42, R43, R44, R5, R6, R7, R8, R9: footprint Resistor_SMD:R_0805_2012Metric_Pad1.15x1.40mm_HandSolder -> Resistor_SMD:R_0603_1608Metric_Pad1.05x0.95mm_HandSolder
- R20, R25, R31: footprint Resistor_SMD:R_0805_2012Metric_Pad1.15x1.40mm_HandSolder -> Potentiometer_SMD:Potentiometer_Vishay_TS53YJ_Vertical
